Commit message: working camera working camera :q

File: lunabotics_sim/urdf/lunabot.urdf.xacro (robot description, xacro)
@@ -97,4 +97,69 @@
   <xacro:wheel prefix="rear_left"   x_reflect="-1" y_reflect="1"/>
   <xacro:wheel prefix="rear_right"  x_reflect="-1" y_reflect="-1"/>
+  <!-- ===================== RGB-D Camera (RealSense-style) ===================== -->
+  <!-- Mounted top-middle of the chassis, facing forward (+X), simulating a
+       RealSense D435-style depth camera: RGB image + depth image + point
+       cloud, all published together. -->
+  <xacro:property name="camera_mount_height" value="0.02"/>
+  <link name="camera_link">
+    <visual>
+      <origin xyz="0 0 0" rpy="0 0 0"/>
+      <geometry>
+        <box size="0.025 0.09 0.025"/>
+      </geometry>
+      <material name="wheel_black"/>
+    </visual>
+    <collision>
+      <origin xyz="0 0 0" rpy="0 0 0"/>
+      <geometry>
+        <box size="0.025 0.09 0.025"/>
+      </geometry>
+    </collision>
+    <inertial>
+      <mass value="0.072"/>
+      <xacro:box_inertia mass="0.072" x="0.025" y="0.09" z="0.025"/>
+    </inertial>
+  </link>
+  <joint name="chassis_to_camera" type="fixed">
+    <parent link="chassis_link"/>
+    <child link="camera_link"/>
+    <!-- top-middle of chassis, facing forward -->
+    <origin xyz="0 0 ${chassis_height/2 + camera_mount_height}" rpy="0 0 0"/>
+  </joint>
+  <!-- Optical frame: camera/ROS convention (Z-forward, X-right, Y-down) is
+       rotated relative to the link's URDF convention (X-forward, Z-up). -->
+  <link name="camera_optical_link"/>
+  <joint name="camera_to_optical" type="fixed">
+    <parent link="camera_link"/>
+    <child link="camera_optical_link"/>
+    <origin xyz="0 0 0" rpy="-1.5707963267948966 0 -1.5707963267948966"/>
+  </joint>
+  <gazebo reference="camera_link">
+    <sensor name="realsense_depth_camera" type="rgbd_camera">
+      <always_on>true</always_on>
+      <update_rate>30</update_rate>
+      <visualize>true</visualize>
+      <topic>camera</topic>
+      <camera>
+        <optical_frame_id>camera_optical_link</optical_frame_id>
+        <horizontal_fov>1.211</horizontal_fov>
+        <image>
+          <width>640</width>
+          <height>480</height>
+          <format>R8G8B8</format>
+        </image>
+        <clip>
+          <near>0.1</near>
+          <far>50</far>
+        </clip>
+        <depth_camera>
+          <clip>
+            <near>0.1</near>
+            <far>10.0</far>
+          </clip>
+        </depth_camera>
+      </camera>
+    </sensor>
+  </gazebo>
   <!-- ===================== Gazebo plugins ===================== -->
   <!-- Joint-state publishing (so /joint_states is available) plus a

Commit message: added a pillar to robot udrf for testing. Preliminary code for CV

File: lunabotics_sim/urdf/lunabot.urdf.xacro (robot description, xacro)
@@ -17,4 +17,12 @@
   <xacro:property name="wheel_y_offset" value="${chassis_width/2 + wheel_width/2}"/>
   <xacro:property name="wheel_z_offset" value="0.0"/>
+  <!-- Camera mast: raises the RGB-D camera above the chassis for a better
+       vantage point, and tilts it downward to look at terrain ahead. -->
+  <xacro:property name="mast_radius" value="0.015"/>
+  <xacro:property name="mast_height" value="0.15"/>
+  <xacro:property name="mast_mass"   value="0.05"/>
+  <!-- Positive rotation about Y tilts the link's +X (forward) axis toward
+       -Z (downward) in this X-forward/Z-up convention. ~20 degrees. -->
+  <xacro:property name="camera_tilt" value="0.3491"/>
   <material name="chassis_grey">
     <color rgba="0.6 0.6 0.6 1.0"/>
@@ -97,6 +105,35 @@
   <xacro:wheel prefix="rear_left"   x_reflect="-1" y_reflect="1"/>
   <xacro:wheel prefix="rear_right"  x_reflect="-1" y_reflect="-1"/>
+  <!-- ===================== Camera mast ===================== -->
+  <!-- Vertical cylindrical post that raises the camera above the chassis
+       deck for a better vantage point over the terrain ahead. -->
+  <link name="camera_mast_link">
+    <visual>
+      <origin xyz="0 0 0" rpy="0 0 0"/>
+      <geometry>
+        <cylinder radius="${mast_radius}" length="${mast_height}"/>
+      </geometry>
+      <material name="wheel_black"/>
+    </visual>
+    <collision>
+      <origin xyz="0 0 0" rpy="0 0 0"/>
+      <geometry>
+        <cylinder radius="${mast_radius}" length="${mast_height}"/>
+      </geometry>
+    </collision>
+    <inertial>
+      <mass value="${mast_mass}"/>
+      <xacro:cylinder_inertia mass="${mast_mass}" r="${mast_radius}" h="${mast_height}"/>
+    </inertial>
+  </link>
+  <joint name="chassis_to_mast" type="fixed">
+    <parent link="chassis_link"/>
+    <child link="camera_mast_link"/>
+    <!-- mast base sits flush on top of the chassis; mast_link origin is its
+         own center, so raise by half the chassis height plus half the mast -->
+    <origin xyz="0 0 ${chassis_height/2 + mast_height/2}" rpy="0 0 0"/>
+  </joint>
   <!-- ===================== RGB-D Camera (RealSense-style) ===================== -->
-  <!-- Mounted top-middle of the chassis, facing forward (+X), simulating a
+  <!-- Mounted on top of the mast, tilted downward, simulating a
        RealSense D435-style depth camera: RGB image + depth image + point
        cloud, all published together. -->
@@ -121,9 +158,9 @@
     </inertial>
   </link>
-  <joint name="chassis_to_camera" type="fixed">
-    <parent link="chassis_link"/>
+  <joint name="mast_to_camera" type="fixed">
+    <parent link="camera_mast_link"/>
     <child link="camera_link"/>
-    <!-- top-middle of chassis, facing forward -->
-    <origin xyz="0 0 ${chassis_height/2 + camera_mount_height}" rpy="0 0 0"/>
+    <!-- top of the mast, tilted downward by camera_tilt about Y -->
+    <origin xyz="0 0 ${mast_height/2 + camera_mount_height}" rpy="0 ${camera_tilt} 0"/>
   </joint>
   <!-- Optical frame: camera/ROS convention (Z-forward, X-right, Y-down) is

Commit message: changed camera angle back and move robot to face fiducial marker

File: lunabotics_sim/urdf/lunabot.urdf.xacro (robot description, xacro)
@@ -17,4 +17,12 @@
   <xacro:property name="wheel_y_offset" value="${chassis_width/2 + wheel_width/2}"/>
   <xacro:property name="wheel_z_offset" value="0.0"/>
+  <!-- Camera mast: raises the RGB-D camera above the chassis for a better
+       vantage point, and tilts it downward to look at terrain ahead. -->
+  <xacro:property name="mast_radius" value="0.015"/>
+  <xacro:property name="mast_height" value="0.15"/>
+  <xacro:property name="mast_mass"   value="0.05"/>
+  <!-- Positive rotation about Y tilts the link's +X (forward) axis toward
+       -Z (downward) in this X-forward/Z-up convention. ~20 degrees. -->
+  <xacro:property name="camera_tilt" value="0.3491"/>
   <material name="chassis_grey">
     <color rgba="0.6 0.6 0.6 1.0"/>
@@ -90,13 +98,40 @@
     </inertial>
   </link>
-  <!-- ===================== Wheels (free-rolling, no drivetrain) ===================== -->
-  <!-- continuous joints only — nothing commands them yet. Drivetrain plugin
-       (diff-drive/skid-steer) is a later pass. -->
+  <!-- ===================== Wheels ===================== -->
   <xacro:wheel prefix="front_left"  x_reflect="1"  y_reflect="1"/>
   <xacro:wheel prefix="front_right" x_reflect="1"  y_reflect="-1"/>
   <xacro:wheel prefix="rear_left"   x_reflect="-1" y_reflect="1"/>
   <xacro:wheel prefix="rear_right"  x_reflect="-1" y_reflect="-1"/>
+  <!-- ===================== Camera mast ===================== -->
+  <!-- Vertical cylindrical post that raises the camera above the chassis
+       deck for a better vantage point over the terrain ahead. -->
+  <link name="camera_mast_link">
+    <visual>
+      <origin xyz="0 0 0" rpy="0 0 0"/>
+      <geometry>
+        <cylinder radius="${mast_radius}" length="${mast_height}"/>
+      </geometry>
+      <material name="wheel_black"/>
+    </visual>
+    <collision>
+      <origin xyz="0 0 0" rpy="0 0 0"/>
+      <geometry>
+        <cylinder radius="${mast_radius}" length="${mast_height}"/>
+      </geometry>
+    </collision>
+    <inertial>
+      <mass value="${mast_mass}"/>
+      <xacro:cylinder_inertia mass="${mast_mass}" r="${mast_radius}" h="${mast_height}"/>
+    </inertial>
+  </link>
+  <joint name="chassis_to_mast" type="fixed">
+    <parent link="chassis_link"/>
+    <child link="camera_mast_link"/>
+    <!-- mast base sits flush on top of the chassis; mast_link origin is its
+         own center, so raise by half the chassis height plus half the mast -->
+    <origin xyz="0 0 ${chassis_height/2 + mast_height/2}" rpy="0 0 0"/>
+  </joint>
   <!-- ===================== RGB-D Camera (RealSense-style) ===================== -->
-  <!-- Mounted top-middle of the chassis, facing forward (+X), simulating a
+  <!-- Mounted on top of the mast, tilted downward, simulating a
        RealSense D435-style depth camera: RGB image + depth image + point
        cloud, all published together. -->
@@ -121,9 +156,10 @@
     </inertial>
   </link>
-  <joint name="chassis_to_camera" type="fixed">
-    <parent link="chassis_link"/>
+  <joint name="mast_to_camera" type="fixed">
+    <parent link="camera_mast_link"/>
     <child link="camera_link"/>
-    <!-- top-middle of chassis, facing forward -->
-    <origin xyz="0 0 ${chassis_height/2 + camera_mount_height}" rpy="0 0 0"/>
+    <!-- top of the mast, tilted downward by camera_tilt about Y -->
+    <origin xyz="0 0 ${mast_height/2 + camera_mount_height}" rpy="0 0 0"/>
+    <!-- <origin xyz="0 0 ${mast_height/2 + camera_mount_height}" rpy="0 ${camera_tilt} 0"/> -->
   </joint>
   <!-- Optical frame: camera/ROS convention (Z-forward, X-right, Y-down) is

Commit message: cheated bc it is sim and used real ODOM topic. in the future we will have to correct this!

File: lunabotics_sim/urdf/lunabot.urdf.xacro (robot description, xacro)
@@ -61,5 +61,7 @@
       <inertial>
         <mass value="${wheel_mass}"/>
-        <xacro:cylinder_inertia mass="${wheel_mass}" r="${wheel_radius}" h="${wheel_width}"/>
+        <inertia ixx="${(1/12)*wheel_mass*(3*wheel_radius*wheel_radius + wheel_width*wheel_width)}" ixy="0" ixz="0"
+         iyy="${0.5*wheel_mass*wheel_radius*wheel_radius}" iyz="0"
+         izz="${(1/12)*wheel_mass*(3*wheel_radius*wheel_radius + wheel_width*wheel_width)}"/>
       </inertial>
     </link>
@@ -72,5 +74,5 @@
   </xacro:macro>
   <xacro:property name="steer_limit"  value="0.6"/>  <!-- rad, joint hard limit tune later -->
-  <xacro:macro name="steering_knuckle" params="prefix y_reflect">
+  <!-- <xacro:macro name="steering_knuckle" params="prefix y_reflect">
     <link name="${prefix}_steer_link">
       <inertial>
@@ -78,6 +80,6 @@
         <xacro:box_inertia mass="0.2" x="0.05" y="0.05" z="0.05"/>
       </inertial>
-    </link>
-    <joint name="${prefix}_steer_joint" type="revolute">
+    </link> -->
+    <!-- <joint name="${prefix}_steer_joint" type="revolute">
       <parent link="chassis_link"/>
       <child link="${prefix}_steer_link"/>
@@ -86,5 +88,5 @@
       <limit lower="${-steer_limit}" upper="${steer_limit}" effort="20" velocity="2.0"/>
     </joint>
-  </xacro:macro>
+  </xacro:macro> -->
   <!-- ===================== Base / chassis ===================== -->
   <link name="base_link"/>
@@ -116,8 +118,8 @@
   <!-- ===================== Wheels ===================== -->
    <!-- Front: steered -->
-  <xacro:steering_knuckle prefix="front_left"  y_reflect="1"/>
-  <xacro:steering_knuckle prefix="front_right" y_reflect="-1"/>
-  <xacro:wheel prefix="front_left"  parent="front_left_steer_link"  xyz="0 0 0"/>
-  <xacro:wheel prefix="front_right" parent="front_right_steer_link" xyz="0 0 0"/>
+  <xacro:wheel prefix="front_left"  parent="chassis_link"
+             xyz="${wheel_x_offset} ${wheel_y_offset} ${wheel_z_offset}"/>
+  <xacro:wheel prefix="front_right" parent="chassis_link"
+             xyz="${wheel_x_offset} ${-wheel_y_offset} ${wheel_z_offset}"/>
   <!-- Rear: fixed direction -->
   <xacro:wheel prefix="rear_left"  parent="chassis_link"
@@ -225,5 +227,73 @@
        DiffDrive system plugin so the wheels actually respond to velocity
        commands. 4-wheel skid-steer: two joints per side. -->
-   <gazebo>
+  <xacro:property name="track_factor" value="1.0"/>
+  <xacro:property name="wheel_separation_eff"
+                  value="${(chassis_width + wheel_width) * track_factor}"/>
+    <gazebo>
+    <plugin filename="gz-sim-joint-state-publisher-system"
+            name="gz::sim::systems::JointStatePublisher">
+      <joint_name>front_left_wheel_joint</joint_name>
+      <joint_name>front_right_wheel_joint</joint_name>
+      <joint_name>rear_left_wheel_joint</joint_name>
+      <joint_name>rear_right_wheel_joint</joint_name>
+    </plugin>
+    <plugin filename="gz-sim-diff-drive-system"
+          name="gz::sim::systems::DiffDrive">
+    <left_joint>front_left_wheel_joint</left_joint>
+    <left_joint>rear_left_wheel_joint</left_joint>
+    <right_joint>front_right_wheel_joint</right_joint>
+    <right_joint>rear_right_wheel_joint</right_joint>
+    <wheel_separation>${wheel_separation_eff}</wheel_separation>
+    <wheel_radius>${wheel_radius}</wheel_radius>
+    <topic>/cmd_vel</topic>
+    <max_linear_velocity>1.0</max_linear_velocity>
+    <max_angular_velocity>1.5</max_angular_velocity>
+    <max_linear_acceleration>1.0</max_linear_acceleration>
+    <max_angular_acceleration>2.0</max_angular_acceleration>
+  </plugin>
+    <!-- <plugin filename="gz-sim-diff-drive-system"
+            name="gz::sim::systems::DiffDrive">
+      <left_joint>front_left_wheel_joint</left_joint>
+      <left_joint>rear_left_wheel_joint</left_joint>
+      <right_joint>front_right_wheel_joint</right_joint>
+      <right_joint>rear_right_wheel_joint</right_joint>
+      <wheel_separation>${wheel_separation_eff}</wheel_separation>
+      <wheel_radius>${wheel_radius}</wheel_radius>
+      <topic>/cmd_vel</topic>
+      <odom_topic>/odom</odom_topic>
+      <tf_topic>/tf</tf_topic>
+      <frame_id>odom</frame_id>
+      <child_frame_id>base_link</child_frame_id>
+      <odom_publish_frequency>50</odom_publish_frequency> -->
+      <!-- Smooth commands so wheels don't slip/spin out on start/stop -->
+      <!-- <max_linear_velocity>1.0</max_linear_velocity>
+      <max_angular_velocity>1.5</max_angular_velocity>
+      <max_linear_acceleration>1.0</max_linear_acceleration>
+      <max_angular_acceleration>2.0</max_angular_acceleration>
+    </plugin> -->
+    <plugin filename="gz-sim-odometry-publisher-system"
+          name="gz::sim::systems::OdometryPublisher">
+    <odom_frame>odom</odom_frame>
+    <robot_base_frame>base_link</robot_base_frame>
+    <odom_publish_frequency>50</odom_publish_frequency>
+    <odom_topic>/odom</odom_topic>
+    <tf_topic>/tf</tf_topic>
+    <dimensions>2</dimensions>
+  </plugin>
+  </gazebo>
+    <xacro:macro name="wheel_friction" params="link">
+    <gazebo reference="${link}">
+      <mu1>0.5</mu1>
+      <mu2>0.5</mu2>
+      <kp>1000000.0</kp>
+      <kd>100.0</kd>
+    </gazebo>
+  </xacro:macro>
+  <xacro:wheel_friction link="front_left_wheel_link"/>
+  <xacro:wheel_friction link="front_right_wheel_link"/>
+  <xacro:wheel_friction link="rear_left_wheel_link"/>
+  <xacro:wheel_friction link="rear_right_wheel_link"/>
+   <!-- Ackermann plugin -->
+   <!-- <gazebo>
     <plugin filename="gz-sim-joint-state-publisher-system"
             name="gz::sim::systems::JointStatePublisher">
@@ -235,9 +305,6 @@
       <joint_name>front_right_steer_joint</joint_name>
     </plugin>
-    <!-- 4-Wheel Skid-Steer / Diff Drive Plugin -->
-    <plugin filename="gz-sim-diff-drive-system"
-            name="gz::sim::systems::DiffDrive">
-    <!-- <plugin filename="gz-sim-ackermann-steering-system"
-            name="gz::sim::systems::AckermannSteering"> -->
+    <plugin filename="gz-sim-ackermann-steering-system"
+            name="gz::sim::systems::AckermannSteering">
       <left_joint>front_left_wheel_joint</left_joint>
       <left_joint>rear_left_wheel_joint</left_joint>
@@ -258,4 +325,4 @@
       <odom_publish_frequency>30</odom_publish_frequency>
     </plugin>
-  </gazebo>
+  </gazebo> -->
 </robot>
